Commit message: changed mesh file to fix visualizaiton issue

File: urdf/_d435.urdf.xacro (robot description, xacro)
@@ -67,5 +67,5 @@
         <geometry>
           <!-- <box size="${d435_cam_width} ${d435_cam_height} ${d435_cam_depth}"/> -->
-          <mesh filename="package://realsense2_description/meshes/d435.dae"/>
+          <mesh filename="package://realsense_gazebo_description/meshes/d435.dae"/>
           <!--<mesh filename="package://realsense2_description/meshes/d435/d435.dae"/>-->
         </geometry>

File: urdf/_d435i.urdf.xacro (robot description, xacro)
@@ -70,5 +70,5 @@
         <geometry>
           <!-- <box size="${d435i_cam_width} ${d435i_cam_height} ${d435i_cam_depth}"/> -->
-          <mesh filename="package://realsense2_description/meshes/d435.dae"/>
+          <mesh filename="package://realsense_gazebo_description/meshes/d435.dae"/>
           <!--<mesh filename="package://realsense2_description/meshes/d435/d435.dae"/>-->
         </geometry>
